File: hardware/electronics/kosmos_V3_PCB.kicad_pcb (KiCad board)
At the start: 2 copper layers, 90 x 80.6 mm, 34 parts, among them J1 Raspberry_Pi_2_3, J2 CDE_ESP, J3 FACADE, J5 Conn_01x05_Female, SW1 DROITE, SW2 GAUCHE, SW3 SW_Reed, U1 Horloge_Arduino, U2 relai_Arduino, U3 jauge

Commit message: je sais plus
Parts:
- removed the REF** at (175.8, 78.7)
- removed the REF** at (169.7, 78.7)
- removed the REF** at (122.4, 71.1)
- removed the REF** at (128.5, 71.1)
- removed the REF** at (168.1, 61.0)
- removed the REF** at (145.8, 95.5)
- removed the REF** at (150.4, 61.0)
- removed the REF** at (138.7, 61.0)
- removed the REF** at (141.2, 95.5)
- removed the REF** at (175.8, 61.0)
- removed the REF** at (169.7, 82.8)
- removed the REF** at (175.8, 82.8)
- added ?: , , F.Cu at (167.6, 59.9)
- added ?: , , F.Cu at (140.7, 96.0)
- added ?: , , F.Cu at (169.7, 78.7)
- added ?: , , F.Cu at (146.3, 96.0)
- added ?: , , F.Cu at (120.9, 71.1)
- added ?: , , F.Cu at (127.5, 71.1)
- added ?: , , F.Cu at (175.8, 78.7)
- added ?: , , F.Cu at (169.7, 83.8)
- added ?: , , F.Cu at (175.8, 83.8)
- added REF**: TestPoint_THTPad_D1.5mm_Drill0.7mm, TestPoint:TestPoint_THTPad_D1.5mm_Drill0.7mm, F.Cu at (175.8, 59.9)
- added REF**: TestPoint_THTPad_D1.5mm_Drill0.7mm, TestPoint:TestPoint_THTPad_D1.5mm_Drill0.7mm, F.Cu at (139.2, 60.5)
- added REF**: TestPoint_THTPad_D1.5mm_Drill0.7mm, TestPoint:TestPoint_THTPad_D1.5mm_Drill0.7mm, F.Cu at (150.4, 60.5)
Routing:
- net +5V: track 225.4 -> 232.1 mm
- net +3V3: track 229.1 -> 228.1 mm
