File: hardware/electronics/kosmos_V3_PCB.kicad_sch (KiCad schematic)
At the start: 21 parts, among them J1 Raspberry_Pi_2_3, J2 CDE_ESP, J3 FACADE, J4 12v_conv, J5 Conn_01x05_Female, J6 5v_conv, SW1 DROITE, SW2 GAUCHE, SW3 SW_Reed, U1 Horloge_Arduino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

Commit message: je sais plus
Parts:
- R1, R2: value 220 -> (none); footprint Resistor_THT:R_Axial_DIN0207_L6.3mm_D2.5mm_P10.16mm_Horizontal -> (none)
Changed lines of the file:
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@@
       (effects (font (size 1.27 1.27)) (justify left))
     )
-    (property "Value" "220" (id 1) (at 39.37 160.0199 0)
+    (property "Value" "" (id 1) (at 39.37 160.0199 0)
       (effects (font (size 1.27 1.27)) (justify left))
     )
-    (property "Footprint" "Resistor_THT:R_Axial_DIN0207_L6.3mm_D2.5mm_P10.16mm_Horizontal" (id 2) (at 35.052 158.75 90)
+    (property "Footprint" "" (id 2) (at 35.052 158.75 90)
       (effects (font (size 1.27 1.27)) hide)
     )
@@
       (effects (font (size 1.27 1.27)) (justify left))
     )
-    (property "Value" "220" (id 1) (at 29.21 160.0199 0)
+    (property "Value" "" (id 1) (at 29.21 160.0199 0)
       (effects (font (size 1.27 1.27)) (justify left))
     )
-    (property "Footprint" "Resistor_THT:R_Axial_DIN0207_L6.3mm_D2.5mm_P10.16mm_Horizontal" (id 2) (at 24.892 158.75 90)
+    (property "Footprint" "" (id 2) (at 24.892 158.75 90)
       (effects (font (size 1.27 1.27)) hide)
     )
@@
     )
     (path "/fd312552-d548-4422-8113-1b9ca520626c"
-      (reference "R1") (unit 1) (value "220") (footprint "Resistor_THT:R_Axial_DIN0207_L6.3mm_D2.5mm_P10.16mm_Horizontal")
+      (reference "R1") (unit 1) (value "100") (footprint "Resistor_THT:R_Axial_DIN0207_L6.3mm_D2.5mm_P10.16mm_Horizontal")
     )
     (path "/f495be8c-aa23-4cd3-8a1d-b964bda32bbb"
-      (reference "R2") (unit 1) (value "220") (footprint "Resistor_THT:R_Axial_DIN0207_L6.3mm_D2.5mm_P10.16mm_Horizontal")
+      (reference "R2") (unit 1) (value "140") (footprint "Resistor_THT:R_Axial_DIN0207_L6.3mm_D2.5mm_P10.16mm_Horizontal")
     )
     (path "/39220a33-8dec-43c5-a397-9878d2b9ba0c"
